Commit message: Turned off collisions for the arm, tuned in new arm positions(need to test)

File: manipulation/kinova_description/urdf/kinova_common.xacro (robot description, xacro)
@@ -35,10 +35,11 @@
              </visual>
 	    </xacro:if>
-            <collision>
+<!-- turn off arm collisions -->
+ <!--            <collision>
                 <geometry>
                     <mesh
                         filename="package://kinova_description/meshes/${link_mesh}.dae"/>
                 </geometry>
-            </collision>
+            </collision> -->
 						<xacro:kinova_inertial mesh_no="${mesh_no}"/>
       </link>
@@ -70,5 +71,5 @@
             <visual>
                 <geometry>
-									<box size = "0.00001 0.00001 0.00001"/>
+				    <box size = "0.00001 0.00001 0.00001"/>
                 </geometry>
             </visual>

Commit message: Finally got correct previsit poses, turned off some other minor collisions in kinova_common1

File: manipulation/kinova_description/urdf/kinova_common.xacro (robot description, xacro)
@@ -74,9 +74,9 @@
                 </geometry>
             </visual>
-            <collision>
+<!--             <collision>
                 <geometry>
 									<box size = "0.00001 0.00001 0.20001"/>
                 </geometry>
-            </collision>
+            </collision> -->
         </link>
     </xacro:macro>
