Commit message: changed the collor of the robotic arm to black

File: manipulation/kinova_description/urdf/j2n6s300_standalone.xacro (robot description, xacro)
@@ -22,4 +22,9 @@
       </geometry>
     <!--<material name="Black" /> -->
+          <material
+        name="">
+        <color
+          rgba="0.2 0.2 0.2 1" />
+      </material>
     </visual>
     <collision>

File: manipulation/kinova_description/urdf/kinova_common.xacro (robot description, xacro)
@@ -22,6 +22,8 @@
                         filename="package://kinova_description/meshes/${link_mesh}.dae"/>
                 </geometry>
-                <material name="carbon_fiber">
-                    <color rgba="0.792156862745098 0.819607843137255 0.933333333333333 1" />
+                <material
+                name="">
+                <color
+                rgba="0.2 0.2 0.2 1" />
                 </material>
             </visual>
@@ -33,4 +35,9 @@
                         filename="package://kinova_description/meshes/${ring_mesh}.STL"/>
                 </geometry>
+                <material
+                name="">
+                <color
+                rgba="0.2 0.2 0.2 1" />
+                </material>
              </visual>
 	    </xacro:if>
@@ -73,4 +80,9 @@
 				    <box size = "0.00001 0.00001 0.00001"/>
                 </geometry>
+                <material
+                name="">
+                <color
+                rgba="0.2 0.2 0.2 1" />
+                </material>
             </visual>
 <!--             <collision>
