Commit message: Fixed transformation between end effector and joint 6 to match the transform between camera frame and joint 6

File: manipulation/kinova_description/urdf/j2n6s300.xacro (robot description, xacro)
@@ -108,5 +108,5 @@
     <property name="joint_camera_origin_rpy" value="1.57 -1.57 2.156" />
     <property name="joint_depth_camera_origin_rpy" value="-1.58 0 -1.58" />
-    <property name="joint_end_effector_origin_rpy" value="0.0 0.0 0" />
+    <property name="joint_end_effector_origin_rpy" value="0.092 0.01 2.1552" />
     <xacro:macro name="j2n6s300" params="base_parent prefix:=j2n6s300">
         <xacro:gazebo_config robot_namespace="${prefix}"/>

File: manipulation/kinova_description/urdf/kinova_common.xacro (robot description, xacro)
@@ -59,5 +59,5 @@
         <limit effort="2000" velocity="1" lower="${joint_lower_limit}" upper="${joint_upper_limit}"/>
         <origin xyz="${joint_origin_xyz}" rpy="${joint_origin_rpy}"/>
-        <dynamics damping="0.0" friction="0.0"/>
+        <dynamics damping="0.2" friction="0.0"/>
      </joint>
    <xacro:unless value="${fixed}">
